Commit message: comau urdf file until axis 5 completed

File: urdf/Comau_Racer3.urdf (robot description, URDF)
Before this commit: robot comau_racer3, 2 links, 1 joints
Links:
- added link link2; visual cylinder length=${l_link2} radius=${r_link2}
- added link link3; visual cylinder length=${l_link3} radius=${r_link3}
- added link link4; visual cylinder length=${l_link4} radius=${r_link4}
- added link link5; visual cylinder length=${l_link5} radius=${r_link5}
- link base_link: geometry visual cylinder length=${l_base} radius=${r_link1}
- link link1: geometry visual cylinder length=${l_link1} radius=0.115
Joints:
- added joint link2_to_link1: type revolute, parent link1, child link2, origin xyz=0 0 ${z_link2tolink1}, axis 0 1 0 , limit lower=${minangle_link2} upper=${maxangle_link2} effort=1000.0 velocity=0.5
- added joint link3_to_link2: type revolute, parent link2, child link3, origin xyz=0 0 ${z_link3tolink2} rpy=0 0 ${pi}, axis 0 1 0 , limit lower=${minangle_link3} upper=${maxangle_link3} effort=1000.0 velocity=0.5
- added joint link4_to_link3: type revolute, parent link3, child link4, origin xyz=0 0 0 rpy=${pi} 0 0, axis 0 0 1 , limit lower=${minangle_link4} upper=${maxangle_link4} effort=1000.0 velocity=0.5
- added joint link5_to_link4: type revolute, parent link4, child link5, origin xyz=${x_link5tolink4} 0 ${z_link5tolink4} rpy=${-pi} 0 0, axis 0 1 0, limit lower=${minangle_link5} upper=${maxangle_link5} effort=1000.0 velocity=0.5
- joint link1_to_base: axis (none) -> 0 0 1; limit (none) -> lower=${minangle_link1} upper=${maxangle_link1} effort=1000.0 velocity=0.5; origin xyz=0 0 ${l_link1tobase} -> xyz=0 0 ${z_link1tobase}; type fixed -> revolute

Commit message: all axes implemented, working

File: urdf/Comau_Racer3.urdf (robot description, URDF)
Before this commit: robot comau_racer3, 6 links, 5 joints
Links:
- added link link6; visual cylinder length=${l_link6} radius=${r_link6}
Joints:
- added joint link6_to_link5: type revolute, parent link5, child link6, origin xyz=0 0 ${z_link6tolink5} rpy=0 0 0, axis 0 0 1, limit lower=${minangle_link6} upper=${maxangle_link6} effort=1000.0 velocity=0.5
- joint link5_to_link4: origin xyz=${x_link5tolink4} 0 ${z_link5tolink4} rpy=${-pi} 0 0 -> xyz=${x_link5tolink4} 0 ${z_link5tolink4} rpy=${pi} 0 ${pi}
